File: pcb-pfs154-s08/pcb.sch (KiCad schematic (older format))
At the start: 10 parts, among them J1 BAT-, J2 BAT+, U1 PFS154-S08

Commit message: Update 8-pin Schematic and README.md
Parts:
- TP2: value Probe_PA6 -> Probe_PA3
Changed lines of the file:
@@
 P 6250 3650
 F 0 "TP2" V 6400 3700 50  0000 R CNN
-F 1 "Probe_PA6" V 6350 3800 50  0000 L CNN
+F 1 "Probe_PA3" V 6350 3800 50  0000 L CNN
 F 2 "TestPoint:TestPoint_THTPad_D2.0mm_Drill1.0mm" H 6450 3650 50  0001 C CNN
 F 3 "~" H 6450 3650 50  0001 C CNN

Commit message: Add Package
Parts:
- U1: footprint (none) -> Package_SO:SOP-8_3.9x4.9mm_P1.27mm
Changed lines of the file:
@@
 F 0 "U1" H 5500 3200 50  0000 C CNN
 F 1 "PFS154-S08" H 5500 3800 50  0000 C CNN
-F 2 "" H 5500 3500 50  0001 C CNN
+F 2 "Package_SO:SOP-8_3.9x4.9mm_P1.27mm" H 5500 3500 50  0001 C CNN
 F 3 "" H 5500 3500 50  0001 C CNN
 	1    5500 3500
